Commit message: docs(examples): flatten and enrich xacro examples with a modular diff-drive robot
- Flattened examples/xacro directory structure by removing redundant subfolders.
- Added a comprehensive, modular diff_drive_robot.xacro example.
- Fixed material tags in materials.xacro for standard compliance.
- Updated examples README with accurate API usage and directory structure.
- Verified xacro parsing via URDFParser.parse_xacro.

Signed-off-by: arounamounchili <patouossa.mounchili@gmail.com>

File: examples/xacro/materials.xacro (robot description, xacro)
@@ -1,9 +1,9 @@
 <?xml version="1.0"?>
 <robot xmlns:xacro="http://www.ros.org/wiki/xacro">
-  <xacro:material name="silver">
+  <material name="silver">
     <color rgba="0.75 0.75 0.75 1.0"/>
-  </xacro:material>
-  <xacro:material name="black">
+  </material>
+  <material name="black">
     <color rgba="0.0 0.0 0.0 1.0"/>
-  </xacro:material>
+  </material>
 </robot>
